Commit message: Atualiza configuracoes e launch da navegacao

File: src/robo_urdf_description/urdf/robo_urdf.xacro (robot description, xacro)
@@ -125,5 +125,5 @@
 </link>
 <joint name="Rigido" type="fixed">
-  <origin xyz="0.0 0.0 0.0" rpy="0 3.14159 0"/>
+  <origin xyz="0.21 0.0 0.06" rpy="0 3.14159 0"/>
   <parent link="base_link"/>
   <child link="lidar_link_1"/>
